Commit message: edit: spawn_kortex_robot.launch to include workstation_gpd and planning group param, edit: robot description; lift table to remove gazebo ground collision jitter

File: kortex_move_it_config/gen3_robotiq_2f_85_move_it_config/config/7dof/gen3_robotiq_2f_85.srdf.xacro (robot description, xacro)
@@ -49,4 +49,14 @@
         <joint name="$(arg prefix)joint_6" value="-0.87" />
         <joint name="$(arg prefix)joint_7" value="1.57" />
+    </group_state>
+    <group_state name="retract" group="manipulator_and_endeffector">
+        <joint name="$(arg prefix)joint_1" value="0" />
+        <joint name="$(arg prefix)joint_2" value="-0.35" />
+        <joint name="$(arg prefix)joint_3" value="3.14" />
+        <joint name="$(arg prefix)joint_4" value="-2.54" />
+        <joint name="$(arg prefix)joint_5" value="0" />
+        <joint name="$(arg prefix)joint_6" value="-0.87" />
+        <joint name="$(arg prefix)joint_7" value="1.57" />
+        <joint name="$(arg prefix)finger_joint" value="0" />
     </group_state>
     <group_state name="vertical" group="arm">

Commit message: updating repo minor edits

File: kortex_move_it_config/gen3_robotiq_2f_85_move_it_config/config/7dof/gen3_robotiq_2f_85.srdf.xacro (robot description, xacro)
@@ -19,4 +19,5 @@
     </group>
     <group name="gripper">
+	<link name="$(arg prefix)end_effector_link" />
         <joint name="$(arg prefix)gripper_base_joint" />
         <joint name="$(arg prefix)finger_joint" />
@@ -77,14 +78,46 @@
         <joint name="$(arg prefix)right_outer_knuckle_joint" value="0" />
     </group_state>
+    <group_state name="quarter" group="gripper">
+        <joint name="$(arg prefix)left_inner_finger_joint" value="0.2" />
+        <joint name="$(arg prefix)right_inner_knuckle_joint" value="0.2" />
+        <joint name="$(arg prefix)finger_joint" value="0.2" />
+        <joint name="$(arg prefix)right_inner_finger_joint" value="-0.2" />
+        <joint name="$(arg prefix)left_inner_knuckle_joint" value="0.2" />
+        <joint name="$(arg prefix)right_outer_knuckle_joint" value="0.2" />
+    </group_state>
+    <group_state name="third" group="gripper">
+        <joint name="$(arg prefix)left_inner_finger_joint" value="0.3" />
+        <joint name="$(arg prefix)right_inner_knuckle_joint" value="0.3" />
+        <joint name="$(arg prefix)finger_joint" value="0.3" />
+        <joint name="$(arg prefix)right_inner_finger_joint" value="-0.3" />
+        <joint name="$(arg prefix)left_inner_knuckle_joint" value="0.3" />
+        <joint name="$(arg prefix)right_outer_knuckle_joint" value="0.3" />
+    </group_state>
+    <group_state name="three_eigths" group="gripper">
+        <joint name="$(arg prefix)left_inner_finger_joint" value="0.3" />
+        <joint name="$(arg prefix)right_inner_knuckle_joint" value="0.3" />
+        <joint name="$(arg prefix)finger_joint" value="0.3" />
+        <joint name="$(arg prefix)right_inner_finger_joint" value="-0.3" />
+        <joint name="$(arg prefix)left_inner_knuckle_joint" value="0.3" />
+        <joint name="$(arg prefix)right_outer_knuckle_joint" value="0.3" />
+    </group_state>
+    <group_state name="half" group="gripper">
+        <joint name="$(arg prefix)left_inner_finger_joint" value="0.4" />
+        <joint name="$(arg prefix)right_inner_knuckle_joint" value="0.4" />
+        <joint name="$(arg prefix)finger_joint" value="0.4" />
+        <joint name="$(arg prefix)right_inner_finger_joint" value="-0.4" />
+        <joint name="$(arg prefix)left_inner_knuckle_joint" value="0.4" />
+        <joint name="$(arg prefix)right_outer_knuckle_joint" value="0.4" />
+    </group_state>
     <group_state name="closed" group="gripper">
-        <joint name="$(arg prefix)left_inner_finger_joint" value="0.8" />
-        <joint name="$(arg prefix)right_inner_knuckle_joint" value="0.8" />
-        <joint name="$(arg prefix)finger_joint" value="0.8" />
-        <joint name="$(arg prefix)right_inner_finger_joint" value="-0.8" />
-        <joint name="$(arg prefix)left_inner_knuckle_joint" value="0.8" />
-        <joint name="$(arg prefix)right_outer_knuckle_joint" value="0.8" />
+        <joint name="$(arg prefix)left_inner_finger_joint" value="0.78" />
+        <joint name="$(arg prefix)right_inner_knuckle_joint" value="0.78" />
+        <joint name="$(arg prefix)finger_joint" value="0.78" />
+        <joint name="$(arg prefix)right_inner_finger_joint" value="-0.78" />
+        <joint name="$(arg prefix)left_inner_knuckle_joint" value="0.78" />
+        <joint name="$(arg prefix)right_outer_knuckle_joint" value="0.78" />
     </group_state>
     <!--END EFFECTOR: Purpose: Represent information about an end effector.-->
-    <end_effector name="robotiq_2f_85" parent_link="$(arg prefix)end_effector_link" group="gripper" parent_group="arm" />
+    <end_effector name="end_effector" parent_link="$(arg prefix)end_effector_link" group="gripper" parent_group="arm" />
     <!--PASSIVE JOINT: Purpose: this element is used to mark joints that are not actuated-->
     <passive_joint name="$(arg prefix)left_inner_finger_joint" />
